File: fw13-LoRa-module.kicad_pcb (KiCad board)
At the start: 2 copper layers, 29 parts, among them J1 USB_B_Micro, J2 Conn_01x02, U1 NCP1117-3.3_SOT223, U2 W25Q128JVS, U3 RP2040, U4 Value, Y1 ABM8-272-T3

Commit message: USB C base
Parts:
- removed J1: USB_B_Micro, RP2040_minimal:USB_Micro-B_Amphenol_10103594-0001LF_Horizontal_modified
- added C18: 100n, Capacitor_SMD:C_0402_1005Metric, F.Cu at (127.5, 84.0)
- moved U4 44.2 mm to (94.2, 114.4), turned to 90 degrees
- moved C1 15.9 mm to (119.4, 65.5)
- moved C17 15.9 mm to (96.6, 67.0)
- moved C5 15.9 mm to (107.7, 71.8)
- moved J2 15.9 mm to (102.6, 65.5)
- moved R1 15.9 mm to (102.5, 71.3)
- moved R2 15.9 mm to (101.0, 71.3)
- moved U1 15.9 mm to (119.5, 71.8)
- moved C4 14.9 mm to (119.5, 78.5)
- moved U2 8.68 mm to (87.0, 93.5)
Connections:
- U3 pad 11: /GPIO8 -> /CS
- U3 pad 12: /GPIO9 -> /DIO1
- U3 pad 14: /GPIO11 -> /RST
- U3 pad 15: /GPIO12 -> /BUSY
- U3 pad 2: /GPIO0 -> /MISO
- U3 pad 4: /GPIO2 -> /SCK
- U3 pad 5: /GPIO3 -> /MOSI
- U4 pad 10: unconnected-(U4-GND2-Pad10) -> GND
- U4 pad 11: unconnected-(U4-BUSY-Pad11) -> /BUSY
- U4 pad 12: unconnected-(U4-DIO1-Pad12) -> /DIO1
- U4 pad 2: unconnected-(U4-MISO-Pad2) -> /MISO
- U4 pad 3: unconnected-(U4-MOSI-Pad3) -> /MOSI
- U4 pad 4: unconnected-(U4-SCK-Pad4) -> /SCK
- U4 pad 5: unconnected-(U4-RST-Pad5) -> /RST
- U4 pad 6: unconnected-(U4-NSS-Pad6) -> /CS
- U4 pad 7: unconnected-(U4-GND1-Pad7) -> GND
- U4 pad 8: unconnected-(U4-VCC-Pad8) -> +3V3
Routing:
- net GND: vias 22 -> 17
- removed copper zone on F.Cu, net VBUS
Other:
- board outline added: 26 x 30 mm

Commit message: USB C base
Parts:
- added P1: USB_C_Plug_USB2.0, Connector_USB:USB_C_Plug_Molex_105444, F.Cu at (94.6, 86.1)
- added R6: 5.1k, Resistor_SMD:R_0603_1608Metric, F.Cu at (88.0, 81.5)

Commit message: AAAAAAAA
Parts:
- removed R6: 5.1k, Resistor_SMD:R_0603_1608Metric
- added D1: LED, LED_SMD:LED_0805_2012Metric, F.Cu at (82.5, 96.5)
- added D2: LED, LED_SMD:LED_0805_2012Metric, F.Cu at (82.5, 99.5)
- added R7: 5.1k, Resistor_SMD:R_0402_1005Metric, F.Cu at (58.7, 89.9)
- added R8: 270, Resistor_SMD:R_0402_1005Metric, F.Cu at (87.3, 97.0)
- added R9: 270, Resistor_SMD:R_0402_1005Metric, F.Cu at (87.3, 99.0)
- P1: footprint Connector_USB:USB_C_Plug_Molex_105444 -> fw13-LoRa-module:USB_C_Plug_Molex_105444
- U1: value NCP1117-3.3_SOT223 -> AMS1117-3.3
- moved C12 37.6 mm to (68.9, 100.4)
- moved C11 36.9 mm to (56.6, 96.3)
- moved C13 36.9 mm to (56.6, 100.5)
- moved C14 36.9 mm to (63.5, 105.8)
- moved C2 36.9 mm to (61.8, 108.8)
- moved U3 36.9 mm to (63.1, 99.3)
- moved Y1 36.9 mm to (63.1, 111.6)
- moved C10 36.9 mm to (67.1, 92.8)
- moved C15 36.9 mm to (69.6, 95.3)
- moved C16 36.9 mm to (69.6, 93.9)
- moved C3 36.9 mm to (64.4, 108.8)
- moved C7 36.9 mm to (64.6, 105.8)
- moved C8 36.9 mm to (66.1, 92.8)
- moved R3 36.9 mm to (64.1, 92.8)
- moved R4 36.9 mm to (65.1, 92.8)
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Connections:
- P1 pad A6: /USB_DP -> /USB_D+
- P1 pad A7: /USB_DN -> /USB_D-
- P1 pad S1: GND -> (no net)
- U3 pad 7: /GPIO5 -> /STATUS
Routing:
- net GND: vias 17 -> 11
- net +3V3: vias 2 -> 0
Other:
- outline, holes or cut-outs redrawn

Commit message: AAAAAAAA
Parts:
- C1, C17, C4: footprint Capacitor_SMD:C_0805_2012Metric -> Capacitor_SMD:C_0603_1608Metric
- C10, C11, C12, C13, C14, C15, C16, C18, C2, C3, C5, C6, C7, C8, C9: footprint Capacitor_SMD:C_0402_1005Metric -> Capacitor_SMD:C_0603_1608Metric
- R1, R2, R3, R4, R5, R7, R8, R9: footprint Resistor_SMD:R_0402_1005Metric -> Resistor_SMD:R_0603_1608Metric
- moved C15 1.61 mm to (69.7, 96.9)
- moved C6 1.50 mm to (60.6, 92.8)
- moved C16 1.40 mm to (69.7, 95.3)
- moved C9 1.00 mm to (62.1, 92.8)
- moved C10 0.99 mm to (68.1, 92.8)
- moved R3 0.51 mm to (63.6, 92.8)
- moved C8 0.49 mm to (66.6, 92.8)
- moved R5 0.44 mm to (62.0, 105.8)
- moved C7 0.40 mm to (65.0, 105.8)
- moved C2 0.20 mm to (61.6, 108.8)
- moved C3 0.19 mm to (64.6, 108.8)
Routing:
- net GND: vias 11 -> 10
- net +3V3: vias 0 -> 1
- net +1V1: vias 4 -> 3

Commit message: trails base
Parts:
- C1, C4, U1: moved to B.Cu
- moved C1 63.3 mm to (60.6, 88.9), turned to -90 degrees
- moved C4 59.3 mm to (61.9, 92.3), turned to 180 degrees
- moved U1 41.9 mm to (67.9, 91.7)
- moved U4 38.2 mm to (58.4, 102.3), turned to 180 degrees
- moved R8 21.9 mm to (68.9, 108.8), turned to 90 degrees
- moved D1 20.8 mm to (68.9, 112.1), turned to 90 degrees
- moved R9 19.0 mm to (71.1, 108.8), turned to 90 degrees
- moved D2 17.0 mm to (71.1, 112.1), turned to 90 degrees
- moved C12 0.86 mm to (69.7, 100.3)
- moved C11 0.41 mm to (56.7, 96.7)
- moved C3 0.31 mm to (64.9, 108.8)
- moved C14 0.31 mm to (63.8, 105.8)
- moved C2 0.31 mm to (61.9, 108.8)
- moved R5 0.31 mm to (62.3, 105.8)
- moved Y1 0.31 mm to (63.4, 111.6)
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Connections:
- U3 pad 29: /GPIO18 -> /STATUS
- U3 pad 7: /STATUS -> /GPIO5
Routing:
- net +3V3: track 0.00 -> 70.8 mm, vias 1 -> 6
- net +1V1: track 0.00 -> 16.4 mm, vias 3 -> 4
- net /XIN: track 0.00 -> 12.2 mm
- net VBUS: track 0.00 -> 10.2 mm
- net /USB_D-: track 0.00 -> 8.67 mm
- net /STATUS: track 0.00 -> 8.36 mm
- net /USB_D+: track 0.00 -> 8.10 mm
- net Net-(C3-Pad1): track 0.00 -> 5.11 mm
- net Net-(P1-CC): track 0.00 -> 2.81 mm
- net /XOUT: track 0.00 -> 2.71 mm
- net Net-(U3-USB_DM): track 0.00 -> 2.51 mm
- net Net-(U3-USB_DP): track 0.00 -> 2.45 mm
- net Net-(D2-A): track 0.00 -> 1.63 mm
- net Net-(D1-A): track 0.00 -> 1.61 mm
- net GND: vias 10 -> 17

Commit message: wiring base
Parts:
- C17: moved to B.Cu
- moved R7 40.8 mm to (99.5, 89.8)
- moved C13 40.6 mm to (97.3, 99.9)
- moved C10 40.6 mm to (108.6, 91.9)
- moved C6 40.6 mm to (101.1, 91.9)
- moved C8 40.6 mm to (107.1, 91.9)
- moved C9 40.6 mm to (102.6, 91.9)
- moved R3 40.6 mm to (104.1, 91.9)
- moved R4 40.6 mm to (105.6, 91.9)
- moved C15 40.5 mm to (110.2, 96.8)
- moved C7 40.5 mm to (105.8, 105.7)
- moved D1 40.5 mm to (109.4, 112.1)
- moved D2 40.5 mm to (111.6, 112.1)
- moved C4 40.5 mm to (102.4, 92.2)
- moved P1 40.5 mm to (100.0, 86.2)
- moved R5 40.5 mm to (102.8, 105.7)
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Routing:
- net +3V3: track 70.8 -> 103.5 mm, vias 6 -> 8
- net /DIO1: track 0.00 -> 14.2 mm
- net /BUSY: track 0.00 -> 12.8 mm, vias 0 -> 2
- net /CS: track 0.00 -> 12.2 mm
- net /SCK: track 0.00 -> 9.96 mm
- net /MOSI: track 0.00 -> 8.99 mm
- net /RST: track 0.00 -> 8.94 mm, vias 0 -> 2
- net /MISO: track 0.00 -> 7.76 mm, vias 0 -> 2
- net VBUS: track 10.2 -> 14.9 mm, vias 0 -> 2
- net +1V1: track 16.4 -> 18.9 mm
- net Net-(U3-USB_DP): track 2.45 -> 3.24 mm
- net Net-(U3-USB_DM): track 2.51 -> 3.28 mm
- net /USB_D-: track 8.67 -> 8.01 mm
- net GND: vias 17 -> 29

Commit message: wiring base
Parts:
- moved R1 25.2 mm to (94.5, 95.1), turned to 180 degrees
- moved R2 24.7 mm to (94.2, 97.5), turned to 90 degrees
- moved C1 2.10 mm to (102.4, 89.0)
- moved J2 0.60 mm to (91.1, 96.1), turned to 0 degrees
- moved C5 0.22 mm to (88.5, 99.8)
Routing:
- net /QSPI_SS: track 0.00 -> 20.9 mm
- net /QSPI_SD1: track 0.00 -> 15.6 mm, vias 0 -> 2
- net /QSPI_SD2: track 0.00 -> 15.3 mm
- net +3V3: track 103.5 -> 114.2 mm
- net /QSPI_SD3: track 0.00 -> 10.0 mm
- net /QSPI_SCLK: track 0.00 -> 9.04 mm
- net /QSPI_SD0: track 0.00 -> 8.03 mm
- net /~{USB_BOOT}: track 0.00 -> 3.02 mm
- net VBUS: track 14.9 -> 13.2 mm
- net +1V1: track 18.9 -> 20.3 mm
- net GND: track 0.00 -> 0.05 mm, vias 29 -> 31
Other:
- outline, holes or cut-outs redrawn

Commit message: idfk
Parts:
- added C19: 10u, Capacitor_SMD:C_0603_1608Metric, B.Cu at (100.3, 98.2)
- added C20: 10u, Capacitor_SMD:C_0603_1608Metric, B.Cu at (91.3, 105.0)
- added C21: 10u, Capacitor_SMD:C_0603_1608Metric, B.Cu at (103.2, 102.2)
- added C22: 10u, Capacitor_SMD:C_0603_1608Metric, B.Cu at (103.3, 96.3)
Routing:
- added copper zone on B.Cu, net GND
