File: fw13-LoRa-module.kicad_sch (KiCad schematic)
At the start: 29 parts, among them J1 USB_B_Micro, J2 Conn_01x02, U1 NCP1117-3.3_SOT223, U2 W25Q128JVS, U3 RP2040, U4 Value, Y1 ABM8-272-T3

Commit message: LM2675MX base
Parts:
- removed J1: USB_B_Micro, RP2040_minimal:USB_Micro-B_Amphenol_10103594-0001LF_Horizontal_modified, symbol Connector:USB_B_Micro
- added C18: 100n, Capacitor_SMD:C_0402_1005Metric, symbol Device:C
Connections:
- net +3V3: now also U4.8 (VCC), C18.1
- net GND: now also U4.10 (GND2), U4.7 (GND1), C18.2
- net BUSY: now reaches U4.11 (BUSY)
- net DIO1: now reaches U4.12 (DIO1)
- net MISO: now reaches U4.2 (MISO)
- net MOSI: now reaches U4.3 (MOSI)
- net SCK: now reaches U4.4 (SCK)
- net RST: now reaches U4.5 (RST)
- net CS: now reaches U4.6 (NSS)
- no-connect marks 1 -> 2
Other:
- note removed: "Crystal"
- moved on the sheet: C1, C2, C3, C4, C5, J2, R1, R2, R5, U1, U2, U4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

Commit message: USB C base
Parts:
- added P1: USB_C_Plug_USB2.0, Expansion_Card:USB_C_Plug_Molex_105444, symbol Connector:USB_C_Plug_USB2.0
- added R6: 5.1k, Resistor_SMD:R_0603_1608Metric, symbol Device:R_Small_US
Connections:
- net GPIO0 is gone; now on net MISO: U3.2 (GPIO0)
- net GPIO11 is gone; now on net RST: U3.14 (GPIO11)
- net GPIO12 is gone; now on net BUSY: U3.15 (GPIO12)
- net GPIO2 is gone; now on net SCK: U3.4 (GPIO2)
- net GPIO3 is gone; now on net MOSI: U3.5 (GPIO3)
- net GPIO8 is gone; now on net CS: U3.11 (GPIO8)
- net GPIO9 is gone; now on net DIO1: U3.12 (GPIO9)
- net GND: now also P1.A1 (GND), P1.A12 (GND), P1.B1 (GND), P1.B12 (GND), P1.S1 (SHIELD), R6.2
- net VBUS: now also P1.A4 (VBUS), P1.A9 (VBUS), P1.B4 (VBUS), P1.B9 (VBUS)
- new net: P1.A5 (CC), R6.1
- new net USB_DN: P1.A7 (D-)
- new net USB_DP: P1.A6 (D+)
- no-connect marks 2 -> 3

Commit message: USB C base
Parts:
- P1: footprint Expansion_Card:USB_C_Plug_Molex_105444 -> Connector_USB:USB_C_Plug_Molex_105444
Changed lines of the file:
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@@
 			)
 		)
-		(property "Footprint" "Expansion_Card:USB_C_Plug_Molex_105444"
+		(property "Footprint" "Connector_USB:USB_C_Plug_Molex_105444"
 			(at 146.05 101.6 0)
 			(effects
@@
 		(on_board yes)
 		(dnp no)
-		(property "Reference" "#PWR01"
+		(property "Reference" "#PWR0101"
 			(at 142.24 135.89 0)
 			(effects
@@
 			(project "fw13-LoRa-module"
 				(path "/8c0b3d8b-46d3-4173-ab1e-a61765f77d61"
-					(reference "#PWR01")
+					(reference "#PWR0101")
 					(unit 1)
 				)

Commit message: AAAAAAAA
Parts:
- removed R6: 5.1k, Resistor_SMD:R_0603_1608Metric, symbol Device:R_Small_US
- removed U1: NCP1117-3.3_SOT223, Package_TO_SOT_SMD:SOT-223-3_TabPin2, symbol Regulator_Linear:NCP1117-3.3_SOT223
- added D1, D2: LED, LED_SMD:LED_0805_2012Metric, symbol Device:LED
- added R7: 5.1k, Resistor_SMD:R_0402_1005Metric, symbol Device:R
- added R8, R9: 270, Resistor_SMD:R_0402_1005Metric, symbol Device:R
- added U1: AMS1117-3.3, Package_TO_SOT_SMD:SOT-223-3_TabPin2, symbol Regulator_Linear:AMS1117-3.3
- P1: footprint Connector_USB:USB_C_Plug_Molex_105444 -> fw13-LoRa-module:USB_C_Plug_Molex_105444
Connections:
- net USB_DN is gone; now on net USB_D-: P1.A7 (D-)
- net USB_DP is gone; now on net USB_D+: P1.A6 (D+)
- net +3V3: now also R8.2, U1.2 (VO)
- net GND: now also P1.SH (SHIELD), D1.1 (K), D2.1 (K), R7.1, U1.1 (GND); no longer P1.S1 (SHIELD)
- net VBUS: now also U1.3 (VI)
- net at P1.A5 (CC): now also R7.2
- net GPIO5 renamed STATUS
- net STATUS: now also R9.2
- new net: D2.2 (A), R9.1
- new net: D1.2 (A), R8.1

Commit message: AAAAAAAA
Parts:
- C1, C17, C4: footprint Capacitor_SMD:C_0805_2012Metric -> Capacitor_SMD:C_0603_1608Metric
- C10, C11, C12, C13, C14, C15, C16, C18, C2, C3, C5, C6, C7, C8, C9: footprint Capacitor_SMD:C_0402_1005Metric -> Capacitor_SMD:C_0603_1608Metric
- R1, R2, R3, R4, R5, R7, R8, R9: footprint Resistor_SMD:R_0402_1005Metric -> Resistor_SMD:R_0603_1608Metric
Changed lines of the file:
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@@
 			)
 		)
-		(property "Footprint" "Resistor_SMD:R_0402_1005Metric"
+		(property "Footprint" "Resistor_SMD:R_0603_1608Metric"
 			(at 118.872 166.37 90)
 			(hide yes)
@@
 			)
 		)
-		(property "Footprint" "Resistor_SMD:R_0402_1005Metric"
+		(property "Footprint" "Resistor_SMD:R_0603_1608Metric"
 			(at 116.84 168.402 90)
 			(hide yes)
@@
 			)
 		)
-		(property "Footprint" "Capacitor_SMD:C_0402_1005Metric"
+		(property "Footprint" "Capacitor_SMD:C_0603_1608Metric"
 			(at 166.0652 167.64 0)
 			(hide yes)
@@
 			)
 		)
-		(property "Footprint" "Resistor_SMD:R_0402_1005Metric"
+		(property "Footprint" "Resistor_SMD:R_0603_1608Metric"
 			(at 110.49 56.642 90)
 			(hide yes)
@@
 			)
 		)
-		(property "Footprint" "Resistor_SMD:R_0402_1005Metric"
+		(property "Footprint" "Resistor_SMD:R_0603_1608Metric"
 			(at 110.49 64.262 90)
 			(hide yes)
@@
 			)
 		)
-		(property "Footprint" "Capacitor_SMD:C_0402_1005Metric"
+		(property "Footprint" "Capacitor_SMD:C_0603_1608Metric"
 			(at 89.8652 31.75 0)
 			(hide yes)
@@
 			)
 		)
-		(property "Footprint" "Capacitor_SMD:C_0402_1005Metric"
+		(property "Footprint" "Capacitor_SMD:C_0603_1608Metric"
 			(at 101.2952 31.75 0)
 			(hide yes)
@@
 			)
 		)
-		(property "Footprint" "Capacitor_SMD:C_0402_1005Metric"
+		(property "Footprint" "Capacitor_SMD:C_0603_1608Metric"
 			(at 112.7252 31.75 0)
 			(hide yes)
@@
 			)
 		)
-		(property "Footprint" "Capacitor_SMD:C_0402_1005Metric"
+		(property "Footprint" "Capacitor_SMD:C_0603_1608Metric"
 			(at 124.1552 31.75 0)
 			(hide yes)
@@
 			)
 		)
-		(property "Footprint" "Capacitor_SMD:C_0402_1005Metric"
+		(property "Footprint" "Capacitor_SMD:C_0603_1608Metric"
 			(at 135.5852 31.75 0)
 			(hide yes)
@@
 			)
 		)
-		(property "Footprint" "Capacitor_SMD:C_0402_1005Metric"
+		(property "Footprint" "Capacitor_SMD:C_0603_1608Metric"
 			(at 147.0152 31.75 0)
 			(hide yes)
@@
 			)
 		)
-		(property "Footprint" "Capacitor_SMD:C_0402_1005Metric"
+		(property "Footprint" "Capacitor_SMD:C_0603_1608Metric"
 			(at 158.4452 31.75 0)
 			(hide yes)
@@
 			)
 		)
-		(property "Footprint" "Capacitor_SMD:C_0402_1005Metric"
+		(property "Footprint" "Capacitor_SMD:C_0603_1608Metric"
 			(at 23.8252 31.75 0)
 			(hide yes)
@@
 			)
 		)
-		(property "Footprint" "Capacitor_SMD:C_0402_1005Metric"
+		(property "Footprint" "Capacitor_SMD:C_0603_1608Metric"
 			(at 35.2552 31.75 0)
 			(hide yes)
@@
 			)
 		)
-		(property "Footprint" "Capacitor_SMD:C_0402_1005Metric"
+		(property "Footprint" "Capacitor_SMD:C_0603_1608Metric"
 			(at 35.2552 46.99 0)
 			(hide yes)
@@
 			)
 		)
-		(property "Footprint" "Capacitor_SMD:C_0402_1005Metric"
+		(property "Footprint" "Capacitor_SMD:C_0603_1608Metric"
 			(at 89.8652 46.99 0)
 			(hide yes)
@@
 			)
 		)
-		(property "Footprint" "Capacitor_SMD:C_0805_2012Metric"
+		(property "Footprint" "Capacitor_SMD:C_0603_1608Metric"
 			(at 232.1052 147.32 0)
 			(hide yes)
@@
 			)
 		)
-		(property "Footprint" "Capacitor_SMD:C_0805_2012Metric"
+		(property "Footprint" "Capacitor_SMD:C_0603_1608Metric"
 			(at 267.6652 147.32 0)
 			(hide yes)
@@
 			)
 		)
-		(property "Footprint" "Capacitor_SMD:C_0805_2012Metric"
+		(property "Footprint" "Capacitor_SMD:C_0603_1608Metric"
 			(at 143.2052 57.15 0)
 			(hide yes)
@@
 			)
 		)
-		(property "Footprint" "Resistor_SMD:R_0402_1005Metric"
+		(property "Footprint" "Resistor_SMD:R_0603_1608Metric"
 			(at 166.37 89.662 90)
 			(hide yes)
@@
 			)
 		)
-		(property "Footprint" "Capacitor_SMD:C_0402_1005Metric"
+		(property "Footprint" "Capacitor_SMD:C_0603_1608Metric"
 			(at 35.56 177.4952 0)
 			(hide yes)
@@
 			)
 		)
-		(property "Footprint" "Resistor_SMD:R_0402_1005Metric"
+		(property "Footprint" "Resistor_SMD:R_0603_1608Metric"
 			(at 237.49 118.872 90)
 			(hide yes)
@@
 			)
 		)
-		(property "Footprint" "Resistor_SMD:R_0402_1005Metric"
+		(property "Footprint" "Resistor_SMD:R_0603_1608Metric"
 			(at 237.49 103.632 90)
 			(hide yes)
@@
 			)
 		)
-		(property "Footprint" "Capacitor_SMD:C_0402_1005Metric"
+		(property "Footprint" "Capacitor_SMD:C_0603_1608Metric"
 			(at 196.5452 67.31 0)
 			(hide yes)
@@
 			)
 		)
-		(property "Footprint" "Resistor_SMD:R_0402_1005Metric"
+		(property "Footprint" "Resistor_SMD:R_0603_1608Metric"
 			(at 72.39 184.912 90)
 			(hide yes)
@@
 			)
 		)
-		(property "Footprint" "Capacitor_SMD:C_0402_1005Metric"
+		(property "Footprint" "Capacitor_SMD:C_0603_1608Metric"
 			(at 35.56 187.6552 0)
 			(hide yes)

Commit message: trails base
Connections:
- net GPIO18 is gone; now on net STATUS: U3.29 (GPIO18)
- net STATUS: no longer U3.7 (GPIO5)
- new net GPIO5: U3.7 (GPIO5)
Changed lines of the file:
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@@
 		)
 	)
-	(label "GPIO18"
+	(label "STATUS"
 		(at 110.49 119.38 180)
 		(effects
@@
 		)
 	)
-	(label "STATUS"
+	(label "GPIO5"
 		(at 110.49 86.36 180)
 		(effects

Commit message: idfk
Parts:
- added C19, C20, C21, C22: 10u, Capacitor_SMD:C_0603_1608Metric, symbol Device:C
Connections:
- net +1V1: now also C21.1, C22.1
- net +3V3: now also C19.1, C20.1
- net GND: now also C19.2, C20.2, C21.2, C22.2
Other:
- moved on the sheet: C17, C18, U4
